File: board/MMv3.kicad_sch (KiCad schematic)
At the start: 26 parts, among them J1 9V, J2 DRV8833_L, J3 left_mot, J4 right_mot, J5 DRV8833_R, Q1 DMG2301L, SW1 PWR, SW2 but, U1 DS28E05R+T, U2 LD1117S50TR_SOT223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

Commit message: adapt to BAC standard capability
Parts:
- U3: footprint extraparts:RPi_Pico_SMD -> extraparts:RPi_Pico
Other:
- note removed: "TODO try smaller ones"
Changed lines of the file:
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@@
     (stroke (width 0) (type default) (color 0 0 0 0))
-  )
-  (text "TODO try smaller ones" (at 172.72 105.41 0)
-    (effects (font (size 1.27 1.27)) (justify left bottom))
   )
   (text "Motor Driver" (at 229.87 140.97 0)
@@
     (property "Reference" "U3" (id 0) (at 134.62 67.31 0))
     (property "Value" "RPi_Pico" (id 1) (at 137.16 69.85 0))
-    (property "Footprint" "extraparts:RPi_Pico_SMD" (id 2) (at 137.16 64.77 0)
+    (property "Footprint" "extraparts:RPi_Pico" (id 2) (at 137.16 64.77 0)
       (effects (font (size 1.27 1.27)) hide)
     )
@@
     )
     (path "/00000000-0000-0000-0000-000060d91ab9"
-      (reference "U3") (unit 1) (value "RPi_Pico") (footprint "extraparts:RPi_Pico_SMD")
-    )
-  )
+      (reference "U3") (unit 1) (value "RPi_Pico") (footprint "extraparts:RPi_Pico")
+    )
+  )
